Commit message: Add camera

File: ur_description/urdf/common.gazebo.xacro (robot description, xacro)
@@ -22,3 +22,43 @@
 -->
   </gazebo>
+<!-- camera -->
+  <gazebo reference="camera_link">
+    <sensor type="camera" name="camera1">
+      <update_rate>30.0</update_rate>
+      <camera name="head">
+        <horizontal_fov>1.3962634</horizontal_fov>
+        <image>
+          <width>800</width>
+          <height>800</height>
+          <format>R8G8B8</format>
+        </image>
+        <clip>
+          <near>0.02</near>
+          <far>300</far>
+        </clip>
+        <noise>
+          <type>gaussian</type>
+          <!-- Noise is sampled independently per pixel on each frame.
+               That pixel's noise value is added to each of its color
+               channels, which at that point lie in the range [0,1]. -->
+          <mean>0.0</mean>
+          <stddev>0.007</stddev>
+        </noise>
+      </camera>
+      <plugin name="camera_controller" filename="libgazebo_ros_camera.so">
+        <alwaysOn>true</alwaysOn>
+        <updateRate>0.0</updateRate>
+        <cameraName>camera1</cameraName>
+        <imageTopicName>image_raw</imageTopicName>
+        <cameraInfoTopicName>camera_info</cameraInfoTopicName>
+        <frameName>camera_link</frameName>
+        <hackBaseline>0.07</hackBaseline>
+        <distortionK1>0.0</distortionK1>
+        <distortionK2>0.0</distortionK2>
+        <distortionK3>0.0</distortionK3>
+        <distortionT1>0.0</distortionT1>
+        <distortionT2>0.0</distortionT2>
+      </plugin>
+    </sensor>
+  </gazebo>
 </robot>

File: ur_description/urdf/ur10.urdf.xacro (robot description, xacro)
@@ -276,4 +276,35 @@
       </collision>
     </link>
+<!-- Camera dimentions -->
+    <xacro:property name="camera_link" value="0.05" />
+    <xacro:property name="height_camera" value="0.157"/>
+    <xacro:property name="axel_offset" value="0.05"/>
+    <joint name="camera_joint" type="fixed">
+    <axis xyz="0 1 0" />
+    <origin xyz="${camera_link} 0 ${height_camera - axel_offset*2}" rpy="0 0 0"/>
+    <parent link="wrist_3_link"/>
+    <child link="camera_link"/>
+  </joint>
+  <!-- Camera -->
+  <link name="camera_link">
+    <collision>
+      <origin xyz="0 0 0" rpy="0 0 0"/>
+      <geometry>
+    <box size="${camera_link} ${camera_link} ${camera_link}"/>
+      </geometry>
+    </collision>
+    <visual>
+      <origin xyz="0 0 0" rpy="0 0 0"/>
+      <geometry>
+    <box size="${camera_link} ${camera_link} ${camera_link}"/>
+      </geometry>
+      <material name="red"/>
+    </visual>
+    <inertial>
+      <mass value="1e-5" />
+      <origin xyz="0 0 0" rpy="0 0 0"/>
+      <inertia ixx="1e-6" ixy="0" ixz="0" iyy="1e-6" iyz="0" izz="1e-6" />
+    </inertial>
+  </link>
     <xacro:ur_arm_transmission prefix="${prefix}" />
     <xacro:ur_arm_gazebo prefix="${prefix}" />

Commit message: Add Joy Script and Colision Ground.

File: ur_description/urdf/common.gazebo.xacro (robot description, xacro)
@@ -4,6 +4,6 @@
     <plugin name="ros_control" filename="libgazebo_ros_control.so">
       <!--robotNamespace>/arm_controller</robotNamespace>
-      <robotSimType>gazebo_ros_control/DefaultRobotHWSim</robotSimType>
-      <legacyModeNS>true</legacyModeNS-->
+      <!robotSimType>gazebo_ros_control/DefaultRobotHWSim</robotSimType-->
+      <legacyModeNS>true</legacyModeNS>
     </plugin>
 <!--

File: ur_description/urdf/ur10.urdf.xacro (robot description, xacro)
@@ -179,5 +179,5 @@
       </xacro:unless>
       <xacro:if value="${joint_limited}">
-        <limit lower="${wrist_1_lower_limit}" upper="${wrist_1_upper_limit}" effort="5000.0" velocity="3.2"/>
+        <limit lower="${wrist_1_lower_limit}" upper="${wrist_1_upper_limit}" effort="54.0" velocity="3.2"/>
       </xacro:if>
       <dynamics damping="0.0" friction="0.0"/>

Commit message: Second TAG add.

File: ur_description/urdf/common.gazebo.xacro (robot description, xacro)
@@ -34,5 +34,5 @@
         </image>
         <clip>
-          <near>0.02</near>
+          <near>0.0415</near>
           <far>300</far>
         </clip>

File: ur_description/urdf/ur10.urdf.xacro (robot description, xacro)
@@ -277,11 +277,11 @@
     </link>
 <!-- Camera dimentions -->
-    <xacro:property name="camera_link" value="0.05" />
+    <xacro:property name="camera_link" value="0.02" />
     <xacro:property name="height_camera" value="0.2"/>
     <xacro:property name="axel_offset" value="0.05"/>
     <joint name="camera_joint" type="fixed">
     <axis xyz="0 0 0" />
-    <origin xyz="${camera_link} 0 ${height_camera - axel_offset*2}" rpy="0 0 0"/>
-    <parent link="shoulder_link"/>
+    <origin xyz="0.01 0 0" rpy="3.1415 0 1.5707"/>
+    <parent link="ee_link"/>
     <child link="camera_link"/>
   </joint>
